Commit message: z map

File: roadmaps/adamsmap_gazebo/gazebo/discbot.xacro (robot description, xacro)
@@ -2,7 +2,6 @@
 <robot name="discbot" xmlns:xacro="http://www.ros.org/wiki/xacro">
   <!-- Constants for robot dimensions -->
-  <xacro:property name="PI" value="3.1415926535897931"/>
-  <xacro:property name="base_radius" value=".15" />
-  <xacro:property name="base_height" value=".2" />
+  <xacro:property name="base_radius" value="1.5" />
+  <xacro:property name="base_height" value="2" />
   <!-- Import all Gazebo-customization elements, including Gazebo colors -->
   <xacro:include filename="$(find adamsmap_gazebo)/gazebo/discbot.gazebo" />
@@ -10,5 +9,5 @@
   <link name="base_link">
     <collision>
-      <origin xyz="0 0 0" rpy="0 0 0"/>
+      <origin xyz="0 0 ${base_height}/2" rpy="0 0 0"/>
       <geometry>
         <cylinder radius="${base_radius}" length="${base_height}">
@@ -17,5 +16,5 @@
     </collision>
     <visual>
-      <origin xyz="0 0 0" rpy="0 0 0"/>
+      <origin xyz="0 0 ${base_height}/2" rpy="0 0 0"/>
       <geometry>
         <cylinder radius="${base_radius}" length="${base_height}">
@@ -25,5 +24,5 @@
     </visual>
     <inertial>
-      <origin xyz="0 0 0" rpy="0 0 0"/>
+      <origin xyz="0 0 ${base_height}/2" rpy="0 0 0"/>
       <mass value="1"/>
       <inertia

Commit message: simulating paths in gazebo

File: roadmaps/adamsmap_gazebo/gazebo/discbot.xacro (robot description, xacro)
@@ -2,6 +2,6 @@
 <robot name="discbot" xmlns:xacro="http://www.ros.org/wiki/xacro">
   <!-- Constants for robot dimensions -->
-  <xacro:property name="base_radius" value="1.5" />
-  <xacro:property name="base_height" value="2" />
+  <xacro:property name="base_radius" value="1" />
+  <xacro:property name="base_height" value="1" />
   <!-- Import all Gazebo-customization elements, including Gazebo colors -->
   <xacro:include filename="$(find adamsmap_gazebo)/gazebo/discbot.gazebo" />

Commit message: waiting differently

File: roadmaps/adamsmap_gazebo/gazebo/discbot.xacro (robot description, xacro)
@@ -2,5 +2,5 @@
 <robot name="discbot" xmlns:xacro="http://www.ros.org/wiki/xacro">
   <!-- Constants for robot dimensions -->
-  <xacro:property name="base_radius" value="1" />
+  <xacro:property name="base_radius" value=".5" />
   <xacro:property name="base_height" value="1" />
   <!-- Import all Gazebo-customization elements, including Gazebo colors -->

Commit message: all csvs

File: roadmaps/adamsmap_gazebo/gazebo/discbot.xacro (robot description, xacro)
@@ -2,5 +2,5 @@
 <robot name="discbot" xmlns:xacro="http://www.ros.org/wiki/xacro">
   <!-- Constants for robot dimensions -->
-  <xacro:property name="base_radius" value=".5" />
+  <xacro:property name="base_diameter" value="1" />
   <xacro:property name="base_height" value="1" />
   <!-- Import all Gazebo-customization elements, including Gazebo colors -->
@@ -11,5 +11,5 @@
       <origin xyz="0 0 ${base_height}/2" rpy="0 0 0"/>
       <geometry>
-        <cylinder radius="${base_radius}" length="${base_height}">
+        <cylinder radius="${base_diameter}/2" length="${base_height}">
         </cylinder>
       </geometry>
@@ -18,5 +18,5 @@
       <origin xyz="0 0 ${base_height}/2" rpy="0 0 0"/>
       <geometry>
-        <cylinder radius="${base_radius}" length="${base_height}">
+        <cylinder radius="${base_diameter}/2" length="${base_height}">
         </cylinder>
       </geometry>
